Commit message: Temporarily taking out Gazebo plugins that crash ROS control from the ridgeback and the spinning laser

File: yumi_description/urdf/Grippers/yumi_servo_gripper.xacro (robot description, xacro)
@@ -75,5 +75,5 @@
              effort="${max_gripper_effort}" velocity="${max_gripper_velocity}" />
       <dynamics damping="${gripper_joint_damping}"/>
-      <mimic joint="${name}_joint"/>
+      <!-- <mimic joint="${name}_joint"/> -->
     </joint>
     <link name="${name}_finger_l">
@@ -95,5 +95,5 @@
     </link>
      <!--Extensions -->
-    <xacro:yumi_servo_gripper_gazebo name="${name}" />
+    <!-- <xacro:yumi_servo_gripper_gazebo name="${name}" /> -->
     <xacro:yumi_servo_gripper_transmission name="${name}" hardware_interface="${hardware_interface}"/>
   </xacro:macro>

File: yumi_description/urdf/yumi.xacro (robot description, xacro)
@@ -473,5 +473,5 @@
     </link>
     <!--Extensions -->
-    <xacro:yumi_gazebo name="${name}" />
+    <!-- <xacro:yumi_gazebo name="${name}" /> -->
     <xacro:yumi_transmission name="${name}" hardware_interface="${hardware_interface}"/>
   </xacro:macro>
